Commit message: fix igjen....

File: urdf/turtlebot3_waffle_pi_for_open_manipulator.gazebo.xacro (robot description, xacro)
@@ -136,5 +136,5 @@
 <!--link : https://www.raspberrypi.org/documentation/hardware/camera/-->
   <gazebo reference="camera_rgb_frame">
-    <sensor type="camera" name="Pi Camera">
+    <sensor type="camera" name="pi_camera">
       <always_on>true</always_on>
       <visualize>$(arg camera_visual)</visualize>

File: urdf/turtlebot3_waffle_pi_for_open_manipulator.urdf.xacro (robot description, xacro)
@@ -2,5 +2,9 @@
 <robot name="turtlebot3_waffle_pi_for_open_manipulator" xmlns:xacro="http://ros.org/wiki/xacro">
   <xacro:include filename="$(find tidybot)/urdf/common_properties.xacro"/>
-  <xacro:include filename="$(find tidybot)/urdf/turtlebot3_waffle_pi_for_open_manipulator.gazebo.xacro"/>
+  <!-- <xacro:include filename="$(find tidybot)/urdf/turtlebot3_waffle_pi_for_open_manipulator.gazebo.xacro"/> -->
+  <!-- Uncomment to disable the physics engine! -->
+  <gazebo>
+    <static>true</static>
+  </gazebo>
   <link name="base_footprint"/>
   <joint name="base_joint" type="fixed">
@@ -13,5 +17,5 @@
       <origin xyz="-0.064 0 0.0" rpy="0 0 0"/>
       <geometry>
-        <mesh filename="package://meshes/waffle_pi_base_for_open_manipulator.stl" scale="0.001 0.001 0.001"/>
+        <mesh filename="$(find tidybot)/meshes/waffle_pi_base_for_open_manipulator.stl" scale="0.001 0.001 0.001"/>
       </geometry>
       <material name="light_black"/>
@@ -44,5 +48,5 @@
       <origin xyz="0 0 0" rpy="1.57 0 0"/>
       <geometry>
-        <mesh filename="package://meshes/wheels/left_tire.stl" scale="0.001 0.001 0.001"/>
+        <mesh filename="$(find tidybot)/meshes/wheels/left_tire.stl" scale="0.001 0.001 0.001"/>
       </geometry>
       <material name="dark"/>
@@ -72,5 +76,5 @@
       <origin xyz="0 0 0" rpy="1.57 0 0"/>
       <geometry>
-        <mesh filename="package://meshes/wheels/right_tire.stl" scale="0.001 0.001 0.001"/>
+        <mesh filename="$(find tidybot)/meshes/wheels/right_tire.stl" scale="0.001 0.001 0.001"/>
       </geometry>
       <material name="dark"/>
@@ -145,5 +149,5 @@
       <origin xyz="0 0 0.0" rpy="0 0 0"/>
       <geometry>
-        <mesh filename="package://meshes/sensors/lds.stl" scale="0.001 0.001 0.001"/>
+        <mesh filename="$(find tidybot)/meshes/sensors/lds.stl" scale="0.001 0.001 0.001"/>
       </geometry>
       <material name="dark"/>
