Commit message: Flyttet rundt på filer

File: urdf/robot_description.urdf.xacro (robot description, xacro)
@@ -50,5 +50,5 @@
       <origin xyz="0 0 0" rpy="1.57 0 0"/>
       <geometry>
-        <mesh filename="$(find tidybot)/meshes/wheels/left_tire.stl" scale="0.001 0.001 0.001"/>
+        <mesh filename="$(find tidybot)/meshes/left_tire.stl" scale="0.001 0.001 0.001"/>
       </geometry>
       <material name="dark"/>
@@ -78,5 +78,5 @@
       <origin xyz="0 0 0" rpy="1.57 0 0"/>
       <geometry>
-        <mesh filename="$(find tidybot)/meshes/wheels/right_tire.stl" scale="0.001 0.001 0.001"/>
+        <mesh filename="$(find tidybot)/meshes/right_tire.stl" scale="0.001 0.001 0.001"/>
       </geometry>
       <material name="dark"/>

Commit message: la til arm_base i urdf (ikke ferdig)

File: urdf/robot_description.urdf.xacro (robot description, xacro)
@@ -96,4 +96,33 @@
       </inertial>
   </link>
+  <!-- ##################### ARM BASE ################# -->
+  <joint name="arm_base_joint" type="fixed">
+    <parent link="base_link"/>
+    <child link="arm_base_link"/>
+    <origin xyz="0.0 0.0 0.0" rpy="0 0 0"/>
+    <axis xyz="0 0 0"/>
+  </joint>
+  <link name="arm_base_link">
+    <visual>
+      <origin xyz="0 0 0" rpy="0 0 0"/>
+      <geometry>
+        <mesh filename="$(find tidybot)/meshes/arm_base.stl" scale="0.001 0.001 0.001"/>
+      </geometry>
+      <material name="dark"/>
+    </visual>
+    <collision>
+      <origin xyz="0 0 0" rpy="0 0 0"/>
+      <geometry>
+        <box size="0.0465 0.0285 0.036"/>
+      </geometry>
+    </collision>
+    <inertial>
+      <origin xyz="0 0 0" />
+      <mass value="0" />
+      <inertia ixx="0" ixy="0" ixz="0"
+               iyy="0" iyz="0"
+               izz="0" />
+      </inertial>
+  </link>
     <!-- ##################### CASTERS ################# -->
   <joint name="caster_back_right_joint" type="fixed">

Commit message: diverse endringer

File: urdf/robot_description.urdf.xacro (robot description, xacro)
@@ -2,4 +2,5 @@
 <robot name="turtlebot3_waffle_pi_for_open_manipulator" xmlns:xacro="http://ros.org/wiki/xacro">
   <xacro:include filename="$(find tidybot)/urdf/common_properties.xacro"/>
+  <!-- <xacro:include filename="$(find tidybot)/urdf/robot_control.gazebo.xacro"/> -->
   <!-- <xacro:include filename="$(find tidybot)/urdf/robot_description.gazebo.xacro"/> -->
   <!-- Uncomment to disable the physics engine! -->
@@ -7,4 +8,9 @@
     <static>true</static>
   </gazebo>
+  <!-- PROPERTIES -->
+   <xacro:property name="arm_base_length" value="0.0465" />
+   <xacro:property name="arm_base_width" value="0.0285" />
+   <xacro:property name="arm_base_height" value="0.036" />
+  <!-- ####################### -->
     <!-- ##################### BASE ################# -->
   <link name="base_footprint"/>
@@ -100,10 +106,10 @@
     <parent link="base_link"/>
     <child link="arm_base_link"/>
-    <origin xyz="0.0 0.0 0.0" rpy="0 0 0"/>
+    <origin xyz="0 0.0 -0.036" rpy="0 0 0"/>
     <axis xyz="0 0 0"/>
   </joint>
   <link name="arm_base_link">
     <visual>
-      <origin xyz="0 0 0" rpy="0 0 0"/>
+      <origin xyz="0 0 ${0.0915}" rpy="0 0 0"/>
       <geometry>
         <mesh filename="$(find tidybot)/meshes/arm_base.stl" scale="0.001 0.001 0.001"/>
@@ -112,7 +118,7 @@
     </visual>
     <collision>
-      <origin xyz="0 0 0" rpy="0 0 0"/>
-      <geometry>
-        <box size="0.0465 0.0285 0.036"/>
+      <origin xyz="-0.064 0 ${0.0915+(0.036/2)}" rpy="0 0 0"/>
+      <geometry>
+        <box size="${arm_base_length} ${arm_base_width} ${arm_base_height}"/>
       </geometry>
     </collision>
@@ -182,5 +188,5 @@
       <origin xyz="0 0 0.0" rpy="0 0 0"/>
       <geometry>
-        <mesh filename="$(find tidybot)/meshes/sensors/lds.stl" scale="0.001 0.001 0.001"/>
+        <mesh filename="$(find tidybot)/meshes/lds.stl" scale="0.001 0.001 0.001"/>
       </geometry>
       <material name="dark"/>

Commit message: added joint descriptions to urdf

File: urdf/robot_description.urdf.xacro (robot description, xacro)
@@ -9,7 +9,23 @@
   </gazebo>
   <!-- PROPERTIES -->
-   <xacro:property name="arm_base_length" value="0.0465" />
-   <xacro:property name="arm_base_width" value="0.0285" />
-   <xacro:property name="arm_base_height" value="0.036" />
+  <xacro:property name="base_offset_x" value="-0.064"/>
+  <xacro:property name="base_offset_y" value="0.0"/>
+  <xacro:property name="base_offset_z" value="0.0"/>
+  <xacro:property name="base_length" value="0.266"/>
+  <xacro:property name="base_width" value="0.266"/>
+  <xacro:property name="base_height" value="0.0915"/>
+  <xacro:property name="arm_base_length" value="0.0465"/>
+  <xacro:property name="arm_base_width" value="0.0285"/>
+  <xacro:property name="arm_base_height" value="0.036"/>
+  <xacro:property name="link_offset_x" value="0.02275"/>
+  <xacro:property name="first_link_length" value="0.028"/>
+  <xacro:property name="first_link_width" value="0.038"/>
+  <xacro:property name="first_link_height" value="0.0405"/>
+  <xacro:property name="second_link_length" value="0.024"/>
+  <xacro:property name="second_link_width" value="0.024"/>
+  <xacro:property name="second_link_height" value="0.150"/>
+  <xacro:property name="third_link_length" value="0.024"/>
+  <xacro:property name="third_link_width" value="0.024"/>
+  <xacro:property name="third_link_height" value="0.120"/>
   <!-- ####################### -->
     <!-- ##################### BASE ################# -->
@@ -18,9 +34,9 @@
     <parent link="base_footprint"/>
     <child link="base_link" />
-    <origin xyz="0 0 0.010" rpy="0 0 0"/>
+    <origin xyz="0 0 0" rpy="0 0 0"/>
   </joint>
   <link name="base_link">
     <visual>
-      <origin xyz="-0.064 0 0.0" rpy="0 0 0"/>
+      <origin xyz="-0.064 0 0" rpy="0 0 0"/>
       <geometry>
         <mesh filename="$(find tidybot)/meshes/waffle_pi_base_for_open_manipulator.stl" scale="0.001 0.001 0.001"/>
@@ -106,10 +122,10 @@
     <parent link="base_link"/>
     <child link="arm_base_link"/>
-    <origin xyz="0 0.0 -0.036" rpy="0 0 0"/>
-    <axis xyz="0 0 0"/>
+    <origin xyz="${base_offset_x} 0 ${base_height}" rpy="0 0 0"/>
+    <axis xyz="0 0 1"/>
   </joint>
   <link name="arm_base_link">
     <visual>
-      <origin xyz="0 0 ${0.0915}" rpy="0 0 0"/>
+      <origin xyz="0 0 ${arm_base_height}" rpy="0 0 0"/>
       <geometry>
         <mesh filename="$(find tidybot)/meshes/arm_base.stl" scale="0.001 0.001 0.001"/>
@@ -118,5 +134,5 @@
     </visual>
     <collision>
-      <origin xyz="-0.064 0 ${0.0915+(0.036/2)}" rpy="0 0 0"/>
+      <origin xyz="${base_offset_x} 0 ${base_height + (arm_base_height)/2}" rpy="0 0 0"/>
       <geometry>
         <box size="${arm_base_length} ${arm_base_width} ${arm_base_height}"/>
@@ -125,8 +141,100 @@
     <inertial>
       <origin xyz="0 0 0" />
-      <mass value="0" />
-      <inertia ixx="0" ixy="0" ixz="0"
-               iyy="0" iyz="0"
-               izz="0" />
+      <mass value="0.001" />
+      <inertia ixx="0.001" ixy="0.001" ixz="0.001"
+               iyy="0.001" iyz="0.001"
+               izz="0.001" />
+      </inertial>
+  </link>
+  <!-- ###################### FIRST LINK #####################-->
+  <joint name="first_link_joint" type="continuous">
+    <parent link="arm_base_link"/>
+    <child link="first_link"/>
+    <origin xyz="0 0 ${arm_base_height}" rpy="0 0 0"/>
+    <axis xyz="0 0 1"/>
+  </joint>
+  <link name="first_link">
+    <visual>
+      <origin xyz="0 0 0" rpy="0 0 0"/>
+      <geometry>
+        <mesh filename="$(find tidybot)/meshes/first_link.stl" scale="0.001 0.001 0.001"/>
+      </geometry>
+      <material name="dark"/>
+    </visual>
+    <collision>
+      <origin xyz="0 0 0" rpy="0 0 0"/>
+      <geometry>
+        <box size="${first_link_length} ${first_link_width} ${first_link_height}"/>
+      </geometry>
+    </collision>
+    <inertial>
+      <origin xyz="0 0 0" />
+      <mass value="0.001" />
+      <inertia ixx="0.001" ixy="0.001" ixz="0.001"
+               iyy="0.001" iyz="0.001"
+               izz="0.001" />
+      </inertial>
+  </link>
+  <!-- ##################### SECOND LINK ################# -->
+  <joint name="second_link_joint" type="revolute">
+    <parent link="first_link"/>
+    <child link="second_link"/>
+    <origin xyz="0 0 ${first_link_height}" rpy="0 0 0"/>
+    <axis xyz="0 0 1"/>
+    <limit effort="100" velocity="100" lower="-${pi/2}" upper="${pi/2}"/>
+    <dynamics damping="0.7" friction="1.0"/>
+  </joint>
+  <link name="second_link">
+    <visual>
+      <origin xyz="${link_offset_x} 0 ${second_link_height}" rpy="0 0 ${-pi/2}"/>
+      <geometry>
+        <mesh filename="$(find tidybot)/meshes/bent_link_150.stl" scale="0.001 0.001 0.001"/>
+      </geometry>
+      <material name="dark"/>
+    </visual>
+    <collision>
+      <origin xyz="0 0 ${-(second_link_height)/2 - 0.0195}" rpy="0 0 0"/>
+      <geometry>
+        <box size="${second_link_length} ${second_link_width} 110"/>
+      </geometry>
+    </collision>
+    <inertial>
+      <origin xyz="0 0 0" />
+      <mass value="0.001" />
+      <inertia ixx="0.001" ixy="0.001" ixz="0.001"
+               iyy="0.001" iyz="0.001"
+               izz="0.001" />
+      </inertial>
+  </link>
+  <!-- ##################### THIRD LINK ################# -->
+  <joint name="third_link_joint" type="revolute">
+    <parent link="second_link"/>
+    <child link="third_link"/>
+    <origin xyz="0 0 0" rpy="0 0 0"/>
+    <axis xyz="0 0 1"/>
+    <limit effort="100" velocity="100" lower="-${pi/2}" upper="${pi/2}"/>
+    <dynamics damping="0.7" friction="1.0"/>
+  </joint>
+  <!-- OBS OBS OBS OBS, SJEKK RPY -->
+  <link name="third_link">
+    <visual>
+      <origin xyz="${link_offset_x} 0 ${second_link_height}" rpy="${pi} 0 ${pi/2}"/>
+      <geometry>
+        <mesh filename="$(find tidybot)/meshes/link_120.stl" scale="0.001 0.001 0.001"/>
+      </geometry>
+      <material name="dark"/>
+    </visual>
+    <collision>
+      <origin xyz="0 0 ${-(second_link_height)/2 - 0.0195}" rpy="0 0 0"/>
+      <geometry>
+        <box size="${third_link_length} ${third_link_width} 110"/>
+      </geometry>
+    </collision>
+    <inertial>
+      <origin xyz="0 0 0" />
+      <mass value="0.001" />
+      <inertia ixx="0.001" ixy="0.001" ixz="0.001"
+               iyy="0.001" iyz="0.001"
+               izz="0.001" />
       </inertial>
   </link>
@@ -206,4 +314,5 @@
     </inertial>
   </link>
+<!--
   <joint name="camera_joint" type="fixed">
     <origin xyz="0.073 -0.011 0.084" rpy="0 0 0"/>
@@ -230,4 +339,4 @@
     <child link="camera_rgb_optical_frame"/>
   </joint>
-  <link name="camera_rgb_optical_frame"/>
+  <link name="camera_rgb_optical_frame"/> -->
 </robot>

Commit message: completed visuals

File: urdf/robot_description.urdf.xacro (robot description, xacro)
@@ -1,4 +1,4 @@
 <?xml version="1.0" ?>
-<robot name="turtlebot3_waffle_pi_for_open_manipulator" xmlns:xacro="http://ros.org/wiki/xacro">
+<robot name="tidybot" xmlns:xacro="http://ros.org/wiki/xacro">
   <xacro:include filename="$(find tidybot)/urdf/common_properties.xacro"/>
   <!-- <xacro:include filename="$(find tidybot)/urdf/robot_control.gazebo.xacro"/> -->
@@ -28,4 +28,13 @@
   <xacro:property name="third_link_width" value="0.024"/>
   <xacro:property name="third_link_height" value="0.120"/>
+  <xacro:property name="gripper_base_length" value="0.070"/>
+  <xacro:property name="gripper_base_width" value="0.104"/>
+  <xacro:property name="gripper_base_height" value="0.05825"/>
+  <xacro:property name="finger_length" value="0.072"/>
+  <xacro:property name="finger_width" value="0.016"/>
+  <xacro:property name="finger_height" value="0.0536"/>
+  <xacro:property name="finger_length_to_center" value="0.0395"/>
+  <xacro:property name="finger_origin_offset" value="0.012"/>
+  <xacro:property name="finger_offset_gripper_open" value="0.036"/>
   <!-- ####################### -->
     <!-- ##################### BASE ################# -->
@@ -181,5 +190,5 @@
     <child link="second_link"/>
     <origin xyz="0 0 ${first_link_height}" rpy="0 0 0"/>
-    <axis xyz="0 0 1"/>
+    <axis xyz="0 1 0"/>
     <limit effort="100" velocity="100" lower="-${pi/2}" upper="${pi/2}"/>
     <dynamics damping="0.7" friction="1.0"/>
@@ -211,13 +220,12 @@
     <parent link="second_link"/>
     <child link="third_link"/>
-    <origin xyz="0 0 0" rpy="0 0 0"/>
-    <axis xyz="0 0 1"/>
+    <origin xyz="${link_offset_x} 0 ${second_link_height}" rpy="0 0 0"/>
+    <axis xyz="0 1 0"/>
     <limit effort="100" velocity="100" lower="-${pi/2}" upper="${pi/2}"/>
     <dynamics damping="0.7" friction="1.0"/>
   </joint>
-  <!-- OBS OBS OBS OBS, SJEKK RPY -->
   <link name="third_link">
     <visual>
-      <origin xyz="${link_offset_x} 0 ${second_link_height}" rpy="${pi} 0 ${pi/2}"/>
+      <origin xyz="${third_link_height} 0 0" rpy="0 0 ${pi/2}"/>
       <geometry>
         <mesh filename="$(find tidybot)/meshes/link_120.stl" scale="0.001 0.001 0.001"/>
@@ -228,5 +236,98 @@
       <origin xyz="0 0 ${-(second_link_height)/2 - 0.0195}" rpy="0 0 0"/>
       <geometry>
-        <box size="${third_link_length} ${third_link_width} 110"/>
+        <box size="${third_link_length} ${third_link_width} 0.110"/>
+      </geometry>
+    </collision>
+    <inertial>
+      <origin xyz="0 0 0" />
+      <mass value="0.001" />
+      <inertia ixx="0.001" ixy="0.001" ixz="0.001"
+               iyy="0.001" iyz="0.001"
+               izz="0.001" />
+      </inertial>
+  </link>
+  <!-- ################## GRIPPER BASE ################### -->
+  <joint name="gripper_base_joint" type="revolute">
+    <parent link="third_link"/>
+    <child link="gripper_base"/>
+    <origin xyz="${third_link_height} 0 0" rpy="0 0 0"/>
+    <axis xyz="0 1 0"/>
+    <limit effort="100" velocity="100" lower="-${pi/2}" upper="${pi/2}"/>
+    <dynamics damping="0.7" friction="1.0"/>
+  </joint>
+  <link name="gripper_base">
+    <visual>
+      <origin xyz="0 0 0" rpy="0 0 ${-pi/2}"/>
+      <geometry>
+        <mesh filename="$(find tidybot)/meshes/gripper_base.stl" scale="0.001 0.001 0.001"/>
+      </geometry>
+      <material name="dark"/>
+    </visual>
+    <collision>
+      <origin xyz="0 0 0" rpy="0 0 0"/>
+      <geometry>
+        <box size="0 0 0"/>
+      </geometry>
+    </collision>
+    <inertial>
+      <origin xyz="0 0 0" />
+      <mass value="0.001" />
+      <inertia ixx="0.001" ixy="0.001" ixz="0.001"
+               iyy="0.001" iyz="0.001"
+               izz="0.001" />
+      </inertial>
+  </link>
+  <!-- ################# LEFT FINGER ################# -->
+  <joint name="left_finger_joint" type="prismatic">
+    <parent link="gripper_base"/>
+    <child link="left_finger"/>
+    <origin xyz="${gripper_base_length} ${finger_origin_offset + finger_offset_gripper_open} 0" rpy="0 0 0"/>
+    <axis xyz="0 1 0"/>
+    <limit effort="100" velocity="100" lower="0" upper="${finger_origin_offset + finger_offset_gripper_open}"/>
+    <dynamics damping="0.7" friction="1.0"/>
+  </joint>
+  <link name="left_finger">
+    <visual>
+      <origin xyz="0 0 0" rpy="0 0 0"/>
+      <geometry>
+        <mesh filename="$(find tidybot)/meshes/gripper_finger.stl" scale="0.001 0.001 0.001"/>
+      </geometry>
+      <material name="dark"/>
+    </visual>
+    <collision>
+      <origin xyz="0 0 0" rpy="0 0 0"/>
+      <geometry>
+        <box size="0 0 0"/>
+      </geometry>
+    </collision>
+    <inertial>
+      <origin xyz="0 0 0" />
+      <mass value="0.001" />
+      <inertia ixx="0.001" ixy="0.001" ixz="0.001"
+               iyy="0.001" iyz="0.001"
+               izz="0.001" />
+      </inertial>
+  </link>
+  <!-- ################# RIGHT FINGER ################# -->
+  <joint name="right_finger_joint" type="prismatic">
+    <parent link="gripper_base"/>
+    <child link="right_finger"/>
+    <origin xyz="${gripper_base_length} ${-(finger_origin_offset + finger_offset_gripper_open)} 0" rpy="0 0 0"/>
+    <axis xyz="0 1 0"/>
+    <limit effort="100" velocity="100" lower="${-(finger_origin_offset + finger_offset_gripper_open)}" upper="0"/>
+    <dynamics damping="0.7" friction="1.0"/>
+  </joint>
+  <link name="right_finger">
+    <visual>
+      <origin xyz="0 0 0" rpy="${pi} 0 0"/>
+      <geometry>
+        <mesh filename="$(find tidybot)/meshes/gripper_finger.stl" scale="0.001 0.001 0.001"/>
+      </geometry>
+      <material name="dark"/>
+    </visual>
+    <collision>
+      <origin xyz="0 0 0" rpy="0 0 0"/>
+      <geometry>
+        <box size="0 0 0"/>
       </geometry>
     </collision>
@@ -294,5 +395,5 @@
   <link name="base_scan">
     <visual>
-      <origin xyz="0 0 0.0" rpy="0 0 0"/>
+      <origin xyz="0.02 0 0" rpy="0 0 0"/>
       <geometry>
         <mesh filename="$(find tidybot)/meshes/lds.stl" scale="0.001 0.001 0.001"/>
