Commit message: lagt til collision

File: urdf/robot_control.gazebo.xacro (robot description, xacro)
@@ -1,5 +1,5 @@
 <?xml version="1.0"?>
 <robot>
-    <gazebo reference="JOINT_NAME">
+    <gazebo reference="arm_base_joint">
         <implicitSpringDamper>true</implicitSpringDamper>
     </gazebo>
@@ -7,5 +7,5 @@
         <plugin filename="libgazebo_ros2_control.so" name="gazebo_ros2_control">
             <robot_sim_type>gazebo_ros2_control/GazeboSystem</robot_sim_type>
-            <parameters>$(find PACKAGE_NAME)/config/FILENAME.yaml</parameters>
+            <parameters>$(find tidybot)/config/controller_config.yaml</parameters>
         </plugin>
     </gazebo>

File: urdf/robot_description.urdf.xacro (robot description, xacro)
@@ -3,5 +3,5 @@
   <xacro:include filename="$(find tidybot)/urdf/common_properties.xacro"/>
   <!-- <xacro:include filename="$(find tidybot)/urdf/robot_control.gazebo.xacro"/> -->
-  <!-- <xacro:include filename="$(find tidybot)/urdf/robot_description.gazebo.xacro"/> -->
+  <!-- <xacro:include filename="$(find tidybot)/urdf/robot_description_original.gazebo.xacro"/> -->
   <!-- Uncomment to disable the physics engine! -->
   <gazebo>
@@ -23,6 +23,6 @@
   <xacro:property name="first_link_height" value="0.0405"/>
   <xacro:property name="second_link_length" value="0.024"/>
-  <xacro:property name="second_link_width" value="0.024"/>
-  <xacro:property name="second_link_height" value="0.150"/>
+  <xacro:property name="second_link_width" value="0.170"/>
+  <xacro:property name="second_link_height" value="0.024"/>
   <xacro:property name="third_link_length" value="0.024"/>
   <xacro:property name="third_link_width" value="0.024"/>
@@ -37,4 +37,5 @@
   <xacro:property name="finger_origin_offset" value="0.012"/>
   <xacro:property name="finger_offset_gripper_open" value="0.036"/>
+  <xacro:property name="collision_box_reduction" value="0.02"/>
   <!-- ####################### -->
     <!-- ##################### BASE ################# -->
@@ -43,5 +44,5 @@
     <parent link="base_footprint"/>
     <child link="base_link" />
-    <origin xyz="0 0 0" rpy="0 0 0"/>
+    <origin xyz="0 0 0.03" rpy="0 0 0"/>
   </joint>
   <link name="base_link">
@@ -54,7 +55,7 @@
     </visual>
     <collision>
-      <origin xyz="-0.064 0 0.047" rpy="0 0 0"/>
-      <geometry>
-        <box size="0.266 0.266 0.094"/>
+      <origin xyz="-0.064 0 0.04575" rpy="0 0 0"/>
+      <geometry>
+        <box size="0.266 0.266 0.0915"/>
       </geometry>
     </collision>
@@ -62,10 +63,7 @@
       <origin xyz="0.0 0 0.0" rpy="0 0 0"/>
       <mass value="1.6329594e+00"/>
-      <inertia ixx="1.0" ixy="0.0" ixz="0.0"
-               iyy="1.0" iyz="0.0"
-               izz="1.0" />
-      <!-- <inertia ixx="8.7002718e-03" ixy="-4.7576583e-05" ixz="1.1160499e-04"
+      <inertia ixx="8.7002718e-03" ixy="-4.7576583e-05" ixz="1.1160499e-04"
                iyy="8.6195418e-03" iyz="-3.5422299e-06"
-               izz="1.4612727e-02" />                -->
+               izz="1.4612727e-02" />
     </inertial>
   </link>
@@ -76,4 +74,6 @@
     <origin xyz="0.0 0.144 0.023" rpy="-1.57 0 0"/>
     <axis xyz="0 0 1"/>
+    <limit effort="100" velocity="100"/>
+    <dynamics damping="0.7" friction="0.01"/>
   </joint>
   <link name="wheel_left_link">
@@ -104,4 +104,6 @@
     <origin xyz="0.0 -0.144 0.023" rpy="-1.57 0 0"/>
     <axis xyz="0 0 1"/>
+    <limit effort="100" velocity="100"/>
+    <dynamics damping="0.7" friction="0.1"/>
   </joint>
   <link name="wheel_right_link">
@@ -143,5 +145,5 @@
     </visual>
     <collision>
-      <origin xyz="${base_offset_x} 0 ${base_height + (arm_base_height)/2}" rpy="0 0 0"/>
+      <origin xyz="-0.0120 0 ${arm_base_height / 2}" rpy="0 0 0"/>
       <geometry>
         <box size="${arm_base_length} ${arm_base_width} ${arm_base_height}"/>
@@ -150,8 +152,8 @@
     <inertial>
       <origin xyz="0 0 0" />
-      <mass value="0.001" />
-      <inertia ixx="0.001" ixy="0.001" ixz="0.001"
-               iyy="0.001" iyz="0.001"
-               izz="0.001" />
+      <mass value="0.045438" />
+      <inertia ixx="7196.83" ixy="2.068e-09" ixz="-129.011"
+               iyy="12433.762" iyz="-2.775e-10"
+               izz="11004.658" />
       </inertial>
   </link>
@@ -172,15 +174,15 @@
     </visual>
     <collision>
-      <origin xyz="0 0 0" rpy="0 0 0"/>
-      <geometry>
-        <box size="${first_link_length} ${first_link_width} ${first_link_height}"/>
-      </geometry>
-    </collision>
-    <inertial>
-      <origin xyz="0 0 0" />
-      <mass value="0.001" />
-      <inertia ixx="0.001" ixy="0.001" ixz="0.001"
-               iyy="0.001" iyz="0.001"
-               izz="0.001" />
+      <origin xyz="0 0 ${first_link_height / 2}" rpy="0 0 0"/>
+      <geometry>
+        <box size="${first_link_length - 0.001} ${first_link_width - 0.001} ${first_link_height / 2}"/>
+      </geometry>
+    </collision>
+    <inertial>
+      <origin xyz="0 0 0" />
+      <mass value="0.060172" />
+      <inertia ixx="21477.332" ixy="13.541" ixz="-430.792"
+               iyy="21301.068" iyz="-111.614"
+               izz="12348.458" />
       </inertial>
   </link>
@@ -189,29 +191,29 @@
     <parent link="first_link"/>
     <child link="second_link"/>
-    <origin xyz="0 0 ${first_link_height}" rpy="0 0 0"/>
+    <origin xyz="0 0 ${arm_base_height}" rpy="0 0 0"/>
     <axis xyz="0 1 0"/>
-    <limit effort="100" velocity="100" lower="-${pi/2}" upper="${pi/2}"/>
-    <dynamics damping="0.7" friction="1.0"/>
+    <limit effort="100" velocity="100" lower="${-(pi)}" upper="${pi}"/>
+    <dynamics damping="0.7" friction="0.01"/>
   </joint>
   <link name="second_link">
     <visual>
-      <origin xyz="${link_offset_x} 0 ${second_link_height}" rpy="0 0 ${-pi/2}"/>
-      <geometry>
-        <mesh filename="$(find tidybot)/meshes/bent_link_150.stl" scale="0.001 0.001 0.001"/>
-      </geometry>
-      <material name="dark"/>
-    </visual>
-    <collision>
-      <origin xyz="0 0 ${-(second_link_height)/2 - 0.0195}" rpy="0 0 0"/>
-      <geometry>
-        <box size="${second_link_length} ${second_link_width} 110"/>
-      </geometry>
-    </collision>
-    <inertial>
-      <origin xyz="0 0 0" />
-      <mass value="0.001" />
-      <inertia ixx="0.001" ixy="0.001" ixz="0.001"
-               iyy="0.001" iyz="0.001"
-               izz="0.001" />
+      <origin xyz="0 0 ${second_link_width}" rpy="${-(pi/2)} 0 ${pi/2}"/>
+      <geometry>
+        <mesh filename="$(find tidybot)/meshes/link_170.stl" scale="0.001 0.001 0.001"/>
+      </geometry>
+      <material name="dark"/>
+    </visual>
+    <collision>
+      <origin xyz="0 0 ${second_link_width / 2}" rpy="${pi/2} 0 0"/>
+      <geometry>
+        <box size="${second_link_length} ${second_link_width - 0.04} ${second_link_height}"/>
+      </geometry>
+    </collision>
+    <inertial>
+      <origin xyz="0 0 0" />
+      <mass value="0.112589" />
+      <inertia ixx="3.509e+05" ixy="-61.351" ixz="-1202.759"
+               iyy="3.432e+05" iyz="-36743.271"
+               izz="38079.446" />
       </inertial>
   </link>
@@ -220,8 +222,8 @@
     <parent link="second_link"/>
     <child link="third_link"/>
-    <origin xyz="${link_offset_x} 0 ${second_link_height}" rpy="0 0 0"/>
+    <origin xyz="0 0 ${second_link_width}" rpy="0 0 0"/>
     <axis xyz="0 1 0"/>
-    <limit effort="100" velocity="100" lower="-${pi/2}" upper="${pi/2}"/>
-    <dynamics damping="0.7" friction="1.0"/>
+    <limit effort="100" velocity="100" lower="${-(2*pi/3)}" upper="${2*pi/3}"/>
+    <dynamics damping="0.7" friction="0.01"/>
   </joint>
   <link name="third_link">
@@ -234,15 +236,15 @@
     </visual>
     <collision>
-      <origin xyz="0 0 ${-(second_link_height)/2 - 0.0195}" rpy="0 0 0"/>
-      <geometry>
-        <box size="${third_link_length} ${third_link_width} 0.110"/>
-      </geometry>
-    </collision>
-    <inertial>
-      <origin xyz="0 0 0" />
-      <mass value="0.001" />
-      <inertia ixx="0.001" ixy="0.001" ixz="0.001"
-               iyy="0.001" iyz="0.001"
-               izz="0.001" />
+      <origin xyz="${third_link_height / 2} 0 0" rpy="0 ${pi/2} 0"/>
+      <geometry>
+        <box size="${third_link_length} ${third_link_width} ${third_link_height - collision_box_reduction}"/>
+      </geometry>
+    </collision>
+    <inertial>
+      <origin xyz="0 0 0" />
+      <mass value="0.094954" />
+      <inertia ixx="1.744e+05" ixy="647.52" ixz="-7.071"
+               iyy="22596.123" iyz="-389.804"
+               izz="1.803e+05" />
       </inertial>
   </link>
@@ -254,5 +256,5 @@
     <axis xyz="0 1 0"/>
     <limit effort="100" velocity="100" lower="-${pi/2}" upper="${pi/2}"/>
-    <dynamics damping="0.7" friction="1.0"/>
+    <dynamics damping="0.7" friction="0.01"/>
   </joint>
   <link name="gripper_base">
@@ -265,15 +267,15 @@
     </visual>
     <collision>
-      <origin xyz="0 0 0" rpy="0 0 0"/>
-      <geometry>
-        <box size="0 0 0"/>
-      </geometry>
-    </collision>
-    <inertial>
-      <origin xyz="0 0 0" />
-      <mass value="0.001" />
-      <inertia ixx="0.001" ixy="0.001" ixz="0.001"
-               iyy="0.001" iyz="0.001"
-               izz="0.001" />
+      <origin xyz="${gripper_base_length / 2} 0 0" rpy="0 0 0"/>
+      <geometry>
+        <box size="${gripper_base_length} ${gripper_base_width} ${gripper_base_height}"/>
+      </geometry>
+    </collision>
+    <inertial>
+      <origin xyz="0 0 0" />
+      <mass value="0.102503" />
+      <inertia ixx="42037.078" ixy="0.002" ixz="-0.051"
+               iyy="74712.63" iyz="1902.432"
+               izz="61851.428" />
       </inertial>
   </link>
@@ -296,15 +298,15 @@
     </visual>
     <collision>
-      <origin xyz="0 0 0" rpy="0 0 0"/>
-      <geometry>
-        <box size="0 0 0"/>
-      </geometry>
-    </collision>
-    <inertial>
-      <origin xyz="0 0 0" />
-      <mass value="0.001" />
-      <inertia ixx="0.001" ixy="0.001" ixz="0.001"
-               iyy="0.001" iyz="0.001"
-               izz="0.001" />
+      <origin xyz="${finger_length / 2} ${-((finger_origin_offset / 2) - 0.002)} 0" rpy="0 0 0"/>
+      <geometry>
+        <box size="${finger_length} ${finger_width} ${finger_height}"/>
+      </geometry>
+    </collision>
+    <inertial>
+      <origin xyz="0 0 0" />
+      <mass value="0.02010" />
+      <inertia ixx="4734.61" ixy="700.053" ixz="22.926"
+               iyy="12948.951" iyz="6.405"
+               izz="8977.298" />
       </inertial>
   </link>
@@ -327,15 +329,15 @@
     </visual>
     <collision>
-      <origin xyz="0 0 0" rpy="0 0 0"/>
-      <geometry>
-        <box size="0 0 0"/>
-      </geometry>
-    </collision>
-    <inertial>
-      <origin xyz="0 0 0" />
-      <mass value="0.001" />
-      <inertia ixx="0.001" ixy="0.001" ixz="0.001"
-               iyy="0.001" iyz="0.001"
-               izz="0.001" />
+      <origin xyz="${finger_length / 2} ${(finger_origin_offset / 2) - 0.002} 0" rpy="0 0 0"/>
+      <geometry>
+        <box size="${finger_length} ${finger_width} ${finger_height}"/>
+      </geometry>
+    </collision>
+    <inertial>
+      <origin xyz="0 0 0" />
+      <mass value="0.02010" />
+      <inertia ixx="4734.61" ixy="700.053" ixz="22.926"
+               iyy="12948.951" iyz="6.405"
+               izz="8977.298" />
       </inertial>
   </link>
@@ -395,5 +397,5 @@
   <link name="base_scan">
     <visual>
-      <origin xyz="0.02 0 0" rpy="0 0 0"/>
+      <origin xyz="0.02 0 -0.01" rpy="0 0 0"/>
       <geometry>
         <mesh filename="$(find tidybot)/meshes/lds.stl" scale="0.001 0.001 0.001"/>
@@ -402,7 +404,7 @@
     </visual>
     <collision>
-      <origin xyz="0.015 0 -0.0065" rpy="0 0 0"/>
-      <geometry>
-        <cylinder length="0.0315" radius="0.045"/>
+      <origin xyz="0.032 0 -0.015" rpy="0 0 0"/>
+      <geometry>
+        <cylinder length="0.031" radius="0.05"/>
       </geometry>
     </collision>
