Commit message: la til div for simulering

File: config/backup/robot_description_backup.urdf.xacro (robot description, xacro)
@@ -2,6 +2,6 @@
 <robot name="tidybot" xmlns:xacro="http://ros.org/wiki/xacro">
   <xacro:include filename="$(find tidybot)/urdf/common_properties.xacro"/>
-  <xacro:include filename="$(find tidybot)/urdf/common_macros.xacro"/>
   <xacro:include filename="$(find tidybot)/urdf/robot_control.gazebo.xacro"/>
+  <!-- <xacro:include filename="$(find tidybot)/urdf/robot_description_original.gazebo.xacro"/> -->
   <!-- Uncomment to disable the physics engine! -->
   <!-- <gazebo>
@@ -9,6 +9,4 @@
   </gazebo> -->
   <!-- PROPERTIES -->
-  <xacro:property name="density_pla" value="600"/>
-  <xacro:property name="density_light" value="150"/>
   <xacro:property name="base_offset_x" value="-0.064"/>
   <xacro:property name="base_offset_y" value="0.0"/>
@@ -46,5 +44,5 @@
     <parent link="base_footprint"/>
     <child link="base_link" />
-    <origin xyz="0 0 0.05" rpy="0 0 0"/>
+    <origin xyz="0 0 0.03" rpy="0 0 0"/>
   </joint>
   <link name="base_link">
@@ -62,7 +60,11 @@
       </geometry>
     </collision>
-    <xacro:inertial_box length="0.266" width="0.266" height="0.0915" density="${density_pla}">
-      <origin xyz="-0.064 0 0.04575" rpy="0 0 0"/>
-    </xacro:inertial_box>
+    <inertial>
+      <origin xyz="0.0 0 0.0" rpy="0 0 0"/>
+      <mass value="1.6329594e+00"/>
+      <inertia ixx="8.7002718e-03" ixy="-4.7576583e-05" ixz="1.1160499e-04"
+               iyy="8.6195418e-03" iyz="-3.5422299e-06"
+               izz="1.4612727e-02" />
+    </inertial>
   </link>
     <!-- ##################### WHEELS ################# -->
@@ -72,6 +74,6 @@
     <origin xyz="0.0 0.144 0.023" rpy="-1.57 0 0"/>
     <axis xyz="0 0 1"/>
-    <limit effort="10" velocity="10"/>
-    <dynamics damping="0.7" friction="1"/>
+    <limit effort="100" velocity="10"/>
+    <dynamics damping="0.7" friction="0.1"/>
   </joint>
   <link name="wheel_left_link">
@@ -102,6 +104,6 @@
     <origin xyz="0.0 -0.144 0.023" rpy="-1.57 0 0"/>
     <axis xyz="0 0 1"/>
-    <limit effort="10" velocity="10"/>
-    <dynamics damping="0.7" friction="1"/>
+    <limit effort="100" velocity="10"/>
+    <dynamics damping="0.7" friction="0.1"/>
   </joint>
   <link name="wheel_right_link">
@@ -148,7 +150,11 @@
       </geometry>
     </collision>
-    <xacro:inertial_box length="${arm_base_length}" width="${arm_base_width}" height="${arm_base_height}" density="${density_pla}">
-      <origin xyz="-0.0120 0 ${arm_base_height / 2}" rpy="0 0 0"/>
-    </xacro:inertial_box>
+    <inertial>
+      <origin xyz="0 0 0" />
+      <mass value="0.045438" />
+      <inertia ixx="0.022246769" ixy="-3.359e-16" ixz="-9.84364e-03"
+               iyy="0.033754425" iyz="-4.002e-15"
+               izz="0.017275382" />
+      </inertial>
   </link>
   <!-- ###################### FIRST LINK #####################-->
@@ -158,6 +164,6 @@
     <origin xyz="0 0 ${arm_base_height}" rpy="0 0 0"/>
     <axis xyz="0 0 1"/>
-    <limit effort="100" velocity="100" lower="${-(pi)}" upper="${pi}"/>
-    <dynamics damping="0.7" friction="1"/>
+    <limit effort="100" velocity="100" lower="${-(2*pi)}" upper="${2*pi}"/>
+    <dynamics damping="0.7" friction="0.1"/>
   </joint>
   <link name="first_link">
@@ -175,7 +181,11 @@
       </geometry>
     </collision>
-    <xacro:inertial_box length="${first_link_length - 0.001}" width="${first_link_width - 0.001}" height="${first_link_height / 2}" density="${density_pla}">
-      <origin xyz="0 0 ${first_link_height / 2}" rpy="0 0 0"/>
-    </xacro:inertial_box>
+    <inertial>
+      <origin xyz="0 0 0" />
+      <mass value="0.060172" />
+      <inertia ixx="0.080027617" ixy="7.2e-08" ixz="4.88443e-04"
+               iyy="0.079853221" iyz="7.46091e-04"
+               izz="0.01237546" />
+      </inertial>
   </link>
   <!-- ##################### SECOND LINK ################# -->
@@ -186,5 +196,5 @@
     <axis xyz="0 1 0"/>
     <limit effort="100" velocity="100" lower="${-(pi)}" upper="${pi}"/>
-    <dynamics damping="0.7" friction="1"/>
+    <dynamics damping="0.7" friction="0.1"/>
   </joint>
   <link name="second_link">
@@ -202,7 +212,11 @@
       </geometry>
     </collision>
-    <xacro:inertial_box length="${second_link_length}" width="${second_link_width - 0.04}" height="${second_link_height}" density="${density_pla}">
-      <origin xyz="0 0 ${second_link_width / 2}" rpy="${pi/2} 0 0"/>
-    </xacro:inertial_box>
+    <inertial>
+      <origin xyz="0 0 0" />
+      <mass value="0.113071" />
+      <inertia ixx="0.7624" ixy="-8362.873e-06" ixz="38.222e-06"
+               iyy="24555.216e-06" iyz="694.419e-06"
+               izz="0.7688" />
+      </inertial>
   </link>
   <!-- ##################### THIRD LINK ################# -->
@@ -213,5 +227,5 @@
     <axis xyz="0 1 0"/>
     <limit effort="100" velocity="100" lower="${-(2*pi/3)}" upper="${2*pi/3}"/>
-    <dynamics damping="0.7" friction="1"/>
+    <dynamics damping="0.7" friction="0.1"/>
   </joint>
   <link name="third_link">
@@ -229,7 +243,11 @@
       </geometry>
     </collision>
-    <xacro:inertial_box length="${third_link_length}" width="${third_link_width}" height="${third_link_height - collision_box_reduction}" density="${density_pla}">
-      <origin xyz="${third_link_height / 2} 0 0" rpy="0 ${pi/2} 0"/>
-    </xacro:inertial_box>
+    <inertial>
+      <origin xyz="0 0 0" />
+      <mass value="0.094954" />
+      <inertia ixx="0.3042" ixy="-4760.104e-03" ixz="38.221e-06"
+               iyy="0.022830453" iyz="697.679e-06"
+               izz="0.3104" />
+      </inertial>
   </link>
   <!-- ################## GRIPPER BASE ################### -->
@@ -240,5 +258,5 @@
     <axis xyz="0 1 0"/>
     <limit effort="100" velocity="100" lower="-${pi/2}" upper="${pi/2}"/>
-    <dynamics damping="0.7" friction="1"/>
+    <dynamics damping="0.7" friction="0.1"/>
   </joint>
   <link name="gripper_base">
@@ -256,7 +274,11 @@
       </geometry>
     </collision>
-    <xacro:inertial_box length="${gripper_base_length - 0.01}" width="${gripper_base_width}" height="${gripper_base_height}" density="${density_light}">
-      <origin xyz="${gripper_base_length / 2} 0 0" rpy="0 0 0"/>
-    </xacro:inertial_box>
+    <inertial>
+      <origin xyz="0 0 0" />
+      <mass value="0.102503" />
+      <inertia ixx="0.3017" ixy="1.76e-07" ixz="-2.5e-08"
+               iyy="79281.744e-06" iyz="-35713.616e-06"
+               izz="0.3159" />
+      </inertial>
   </link>
   <!-- ################# LEFT FINGER ################# -->
@@ -267,5 +289,5 @@
     <axis xyz="0 1 0"/>
     <limit effort="100" velocity="100" lower="0" upper="${finger_origin_offset + finger_offset_gripper_open}"/>
-    <dynamics damping="0.7" friction="1"/>
+    <dynamics damping="0.7" friction="0.5"/>
   </joint>
   <link name="left_finger">
@@ -283,7 +305,11 @@
       </geometry>
     </collision>
-    <xacro:inertial_box length="${finger_length}" width="${finger_width}" height="${finger_height}" density="${density_light}">
-      <origin xyz="${finger_length / 2} ${-((finger_origin_offset / 2) - 0.002)} 0" rpy="0 0 0"/>
-    </xacro:inertial_box>
+    <inertial>
+      <origin xyz="0 0 0" />
+      <mass value="0.02010" />
+      <inertia ixx="5415.545e-06" ixy="3374.112e-06" ixz="80.229e-06"
+               iyy="23455.219e-06" iyz="-8.18e-06"
+               izz="20163.876e-06" />
+      </inertial>
   </link>
   <!-- ################# RIGHT FINGER ################# -->
@@ -294,5 +320,5 @@
     <axis xyz="0 1 0"/>
     <limit effort="100" velocity="100" lower="${-(finger_origin_offset + finger_offset_gripper_open)}" upper="0"/>
-    <dynamics damping="0.7" friction="1"/>
+    <dynamics damping="0.7" friction="0.5"/>
   </joint>
   <link name="right_finger">
@@ -310,7 +336,11 @@
       </geometry>
     </collision>
-    <xacro:inertial_box length="${finger_length}" width="${finger_width}" height="${finger_height}" density="${density_light}">
-      <origin xyz="${finger_length / 2} ${-((finger_origin_offset / 2) - 0.002)} 0" rpy="0 0 0"/>
-    </xacro:inertial_box>
+    <inertial>
+      <origin xyz="0 0 0" />
+      <mass value="0.02010" />
+      <inertia ixx="5415.545e-06" ixy="3374.112e-06" ixz="80.229e-06"
+               iyy="23455.219e-06" iyz="-8.18e-06"
+               izz="20163.876e-06" />
+      </inertial>
   </link>
     <!-- ##################### CASTERS ################# -->
@@ -327,7 +357,11 @@
       </geometry>
     </collision>
-    <xacro:inertial_box length="0.030" width="0.009" height="0.020" density="${density_pla}">
-      <origin xyz="0 0.001 0" rpy="0 0 0"/>
-    </xacro:inertial_box>
+    <inertial>
+      <origin xyz="0 0 0" />
+      <mass value="0.005724" />
+      <inertia ixx="467.937e-06" ixy="0.0" ixz="0.0"
+               iyy="229.437e-06" iyz="0.0"
+               izz="620.10e-06" />
+    </inertial>
   </link>
   <joint name="caster_back_left_joint" type="fixed">
@@ -343,7 +377,11 @@
       </geometry>
     </collision>
-    <xacro:inertial_box length="0.030" width="0.009" height="0.020" density="${density_pla}">
-      <origin xyz="0 0.001 0" rpy="0 0 0"/>
-    </xacro:inertial_box>
+    <inertial>
+      <origin xyz="0 0 0" />
+      <mass value="0.005724" />
+      <inertia ixx="467.937e-06" ixy="0.0" ixz="0.0"
+               iyy="229.437e-06" iyz="0.0"
+               izz="620.10e-06" />
+    </inertial>
   </link>
     <!-- ##################### SENSORS ################# -->
@@ -368,5 +406,5 @@
     </visual>
     <collision>
-      <origin xyz="0.032 0 -0.014" rpy="0 0 0"/>
+      <origin xyz="0.032 0 -0.015" rpy="0 0 0"/>
       <geometry>
         <cylinder length="0.031" radius="0.05"/>

File: urdf/robot_control.gazebo.xacro (robot description, xacro)
@@ -1,7 +1,98 @@
 <?xml version="1.0"?>
 <robot>
-    <gazebo reference="arm_base_joint">
+    <!-- ##### Wheels ##### -->
+    <gazebo reference="wheel_left_link">
+        <mu1>10</mu1>
+        <mu2>10</mu2>
+        <kp>500000.0</kp>
+        <kd>10.0</kd>
+        <minDepth>0.001</minDepth>
+        <maxVel>0.05</maxVel>
+        <fdir1>1 0 0</fdir1>
+        <material>Gazebo/FlatBlack</material>
+    </gazebo>
+    <gazebo reference="wheel_right_link">
+        <mu1>10</mu1>
+        <mu2>10</mu2>
+        <kp>500000.0</kp>
+        <kd>10.0</kd>
+        <minDepth>0.001</minDepth>
+        <maxVel>0.05</maxVel>
+        <fdir1>1 0 0</fdir1>
+        <material>Gazebo/FlatBlack</material>
+    </gazebo>
+    <!-- ##### Casters ##### -->
+    <gazebo reference="caster_back_right_link">
+        <mu1>0.1</mu1>
+        <mu2>0.1</mu2>
+        <kp>1000000.0</kp>
+        <kd>100.0</kd>
+        <minDepth>0.001</minDepth>
+        <maxVel>0.05</maxVel>
+        <material>Gazebo/FlatBlack</material>
+    </gazebo>
+    <gazebo reference="caster_back_left_link">
+        <mu1>0.1</mu1>
+        <mu2>0.1</mu2>
+        <kp>1000000.0</kp>
+        <kd>100.0</kd>
+        <minDepth>0.001</minDepth>
+        <maxVel>0.05</maxVel>
+        <material>Gazebo/FlatBlack</material>
+    </gazebo>
+    <gazebo reference="base_link">
+        <material>Gazebo/DarkGrey</material>
+    </gazebo>
+    <gazebo reference="arm_base_link">
+        <material>Gazebo/DarkGrey</material>
+    </gazebo>
+    <gazebo reference="first_link">
+        <material>Gazebo/DarkGrey</material>
+    </gazebo>
+    <gazebo reference="second_link">
+        <material>Gazebo/DarkGrey</material>
+    </gazebo>
+    <gazebo reference="third_link">
+        <material>Gazebo/DarkGrey</material>
+    </gazebo>
+    <gazebo reference="gripper_base">
+        <material>Gazebo/Grey</material>
+    </gazebo>
+    <gazebo reference="left_finger">
+        <material>Gazebo/Grey</material>
+    </gazebo>
+    <gazebo reference="right_finger">
+        <material>Gazebo/Grey</material>
+    </gazebo>
+    <gazebo reference="base_scan">
+        <material>Gazebo/Grey</material>
+    </gazebo>
+    <!-- ##### Arm joints ##### -->
+    <!-- First joint - 360deg continuous joint -->
+    <gazebo reference="first_link_joint">
         <implicitSpringDamper>true</implicitSpringDamper>
     </gazebo>
+    <!-- Second joint - Revolute joint -->
+    <gazebo reference="second_link_joint">
+        <implicitSpringDamper>true</implicitSpringDamper>
+    </gazebo>
+    <!-- Third joint - Revolute joint -->
+    <gazebo reference="third_link_joint">
+        <implicitSpringDamper>true</implicitSpringDamper>
+    </gazebo>
+    <!-- Fourth joint - Revolute joint -->
+    <gazebo reference="gripper_base_joint">
+        <implicitSpringDamper>true</implicitSpringDamper>
+    </gazebo>
+    <!-- Left finger - Prismatic joint -->
+    <gazebo reference="left_finger_joint">
+        <implicitSpringDamper>true</implicitSpringDamper>
+    </gazebo>
+    <!-- Right finger - Prismatic joint -->
+    <gazebo reference="right_finger_joint">
+        <implicitSpringDamper>true</implicitSpringDamper>
+    </gazebo>
+    <!-- ################################  -->
+         <!-- ##### Ros2 control plugin ##### -->
     <gazebo>
         <plugin filename="libgazebo_ros2_control.so" name="gazebo_ros2_control">
@@ -10,13 +101,24 @@
         </plugin>
     </gazebo>
+    <!-- ##################################### -->
+    <!-- ##### Joint command/state interface definitions ##### -->
     <ros2_control name="GazeboSystem" type="system">
         <hardware>
             <plugin>gazebo_ros2_control/GazeboSystem</plugin>
         </hardware>
-        <!--Add joint command/state interface definitions-->
-        <joint name="JOINT_NAME">
+        <joint name="wheel_left_joint">
+            <command_interface name="velocity"/>
+            <state_interface name="velocity"/>
+            <state_interface name="effort"/>
+        </joint>
+        <joint name="wheel_right_joint">
+            <command_interface name="velocity"/>
+            <state_interface name="velocity"/>
+            <state_interface name="effort"/>
+        </joint>
+        <joint name="first_link_joint">
             <command_interface name="position">
-            <param name="min">-${pi/2}</param>
-            <param name="max">${pi/2}</param>
+                <param name="min">-${2*pi}</param>
+                <param name="max">${2*pi}</param>
             </command_interface>
             <state_interface name="position"/>
@@ -24,5 +126,32 @@
             <state_interface name="effort"/>
         </joint>
-        <joint name="gripper_finger_left_joint">
+        <joint name="second_link_joint">
+            <command_interface name="position">
+                <param name="min">-${2*pi/3}</param>
+                <param name="max">${2*pi/3}</param>
+            </command_interface>
+            <state_interface name="position"/>
+            <state_interface name="velocity"/>
+            <state_interface name="effort"/>
+        </joint>
+        <joint name="third_link_joint">
+            <command_interface name="position">
+                <param name="min">-${pi/2}</param>
+                <param name="max">${pi/2}</param>
+            </command_interface>
+            <state_interface name="position"/>
+            <state_interface name="velocity"/>
+            <state_interface name="effort"/>
+        </joint>
+        <joint name="gripper_base_joint">
+            <command_interface name="position">
+                <param name="min">-${pi/2}</param>
+                <param name="max">${pi/2}</param>
+            </command_interface>
+            <state_interface name="position"/>
+            <state_interface name="velocity"/>
+            <state_interface name="effort"/>
+        </joint>
+        <joint name="left_finger_joint">
             <command_interface name="position"/>
             <state_interface name="position"/>
@@ -30,7 +159,7 @@
             <state_interface name="effort"/>
         </joint>
-        <joint name="gripper_finger_right_joint">
-            <param name="mimic">gripper_finger_left_joint</param>
-            <param name="multiplier">1</param>
+        <joint name="right_finger_joint">
+            <param name="mimic">left_finger_joint</param>
+            <param name="multiplier">-1</param>
             <command_interface name="position"/>
             <state_interface name="position"/>
@@ -39,3 +168,29 @@
         </joint>
     </ros2_control>
+    <!-- ##################################### -->
+    <!-- ##### Differential drive controller plugin ##### -->
+    <gazebo>
+        <plugin name="mobile_base_controller" filename="libgazebo_ros_diff_drive.so">
+            <ros>
+                <!-- <namespace>/demo</namespace>
+                <remapping>cmd_vel:=cmd_demo</remapping>
+                <remapping>odom:=odom_demo</remapping> -->
+            </ros>
+            <update_rate>100</update_rate>
+            <!--1 for differential drive; 2 for skid steer drive-->
+            <num_wheel_pairs>1</num_wheel_pairs>
+            <left_joint>wheel_left_joint</left_joint>
+            <right_joint>wheel_right_joint</right_joint>
+            <wheel_separation>0.287</wheel_separation>
+            <wheel_diameter>0.066</wheel_diameter>
+            <max_wheel_torque>10</max_wheel_torque>
+            <max_wheel_acceleration>1</max_wheel_acceleration>
+            <publish_odom>true</publish_odom>
+            <publish_odom_tf>true</publish_odom_tf>
+            <publish_wheel_tf>false</publish_wheel_tf>
+            <odometry_frame>odom</odometry_frame>
+            <robot_base_frame>base_link</robot_base_frame>
+        </plugin>
+    </gazebo>
+    <!-- ##################################### -->
 </robot>
